File: Eagle/Single Side/Sqaure/Square_V01/ws2812_Sqaure.brd (EAGLE design)
At the start: 25.4 x 25.4 mm, 10 parts

Commit message: Latest large panel designes
Other:
- board text added: "C1"
- board text added: "R1"
